File: CE_SolderingPractice/CESP.kicad_pcb (KiCad board)
At the start: 2 copper layers, 56 x 25.4 mm, 11 parts, among them IC1 ATMEGA168-A, J1 CONN16, J2 CONN16, U1 LM741, U2 7805, U3 LM2902N, U4 LM741, U5 TLC274

Commit message: Added back silk screen. Updated gerbers
Other:
- board text added: "Soldering Practice"
Changed lines of the file:
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@@
     (links 35)
     (no_connects 0)
-    (area 157.404999 116.764999 213.562001 142.315001)
+    (area 155.381 115.901612 213.562001 144.632333)
     (thickness 1.6)
-    (drawings 12)
+    (drawings 13)
     (tracks 129)
     (zones 0)
@@
     )
   )
+  (gr_text "Soldering Practice" (at 184.404 118.364) (layer B.SilkS)
+    (effects (font (size 1 1) (thickness 0.25)) (justify mirror))
+  )
   (gr_line (start 163.322 123.825) (end 157.734 123.825) (angle 90) (layer Edge.Cuts) (width 0.508))

Commit message: Added group logo to back silk screen
Parts:
- added VAL: GRP_NAME_BACK, GRP_NAME_BACK, F.Cu at (177.8, 126.2)
