File: benchbudee/Power.sch (KiCad schematic (older format))
At the start: 12 parts, among them P1 CONN_12X2, SW1 SPST

Commit message: New blinky 4 project, mods to blinky and benchbudee for new version
Parts:
- C1, C2, C3: symbol C -> C-RESCUE-benchbudee
Changed lines of the file:
@@
 EESchema Schematic File Version 2
+LIBS:benchbudee-rescue
 LIBS:power
 LIBS:device
@@
 LIBS:memory
 LIBS:xilinx
-LIBS:special
 LIBS:microcontrollers
 LIBS:dsp
@@
 	3200 3000 5750 3000
 $Comp
-L C C2
+L C-RESCUE-benchbudee C2
 U 1 1 52FD1E1E
 P 8900 3700
@@
 $EndComp
 $Comp
-L C C3
+L C-RESCUE-benchbudee C3
 U 1 1 52FD1E2B
 P 8900 4300
@@
 Connection ~ 8900 4000
 $Comp
-L GND #PWR30
+L GND-RESCUE-benchbudee #PWR30
 U 1 1 52FD1E89
 P 8500 4100
@@
 $EndComp
 $Comp
-L GND #PWR20
+L GND-RESCUE-benchbudee #PWR20
 U 1 1 52FD1E98
 P 2050 2800
@@
 	3550 3400 3800 3400
 $Comp
-L GND #PWR23
+L GND-RESCUE-benchbudee #PWR23
 U 1 1 52FD21FF
 P 5050 3600
@@
 $EndComp
 $Comp
-L C C1
+L C-RESCUE-benchbudee C1
 U 1 1 53569E0A
 P 8900 2000
@@
 $EndComp
 $Comp
-L GND #PWR31
+L GND-RESCUE-benchbudee #PWR31
 U 1 1 53569E91
 P 8900 2250
