File: benchbudee/PowerMonitor.sch (KiCad schematic (older format))
At the start: 0 parts

Commit message: Added power monitor module
Parts:
- added JP? (x3): JUMPER, ~, symbol JUMPER
- added R? (x8): R, ~, symbol R
- added R? (x2): RVAR, ~, symbol RVAR
- added U? (x2): LM317, ~, symbol LM317
- added U? (x2): LM7812, ~, symbol LM7812
- added U? (x2): LM324, symbol LM324
Connections:
- new net: R?.1, R?.2, U?.2 (ADJ)
- new net: R?.2, R?.2, U?.2 (ADJ)
- new net +12V: JP?.1, U?.1 (IN), U?.4 (V+), U?.4 (V+), U?.VI
- new net -12V: JP?.2, U?.1 (IN), U?.11 (V-), U?.11 (V-), U?.VI
- new net AGND: JP?.2, R?.1, R?.1, R?.1, R?.2, U?.GND, U?.GND
- new net FE_V+: JP?.2, U?.VO
- new net FE_V-: JP?.1, U?.VO
- new net GND: JP?.1
- new net V+_ADJ: R?.1, R?.1
- new net V+_ADJ_MON: R?.1, R?.2
- new net V+_CURRENT_MON: U?.1, U?.2 (-)
- new net V+_MON: R?.1, R?.2, U?.3 (+), U?.3 (OUT)
- new net V-_ADJ: R?.2, R?.2
- new net V-_ADJ_MON: R?.1, R?.2
- new net V-_CURRENT_MON: U?.1, U?.2 (-)
- new net V-_MON: R?.1, R?.2, U?.3 (+), U?.3 (OUT)

Commit message: Relay module footprints done
Parts:
- gave numbers to parts that had none: 18
Connections:
- net V-_CURRENT_MON: now also U10.6 (-), U10.7; no longer U10.1, U10.2 (-)
- net V-_MON: now also U10.5 (+); no longer U10.3 (+)
Changed lines of the file:
@@
 $EndDescr
 $Comp
-L +3.3V #PWR?
+L +3.3V #PWR031
 U 1 1 52FD5C63
 P 8400 2100
-F 0 "#PWR?" H 8400 2060 30  0001 C CNN
+F 0 "#PWR031" H 8400 2060 30  0001 C CNN
 F 1 "+3.3V" H 8400 2210 30  0000 C CNN
 F 2 "" H 8400 2100 60  0000 C CNN
@@
 $EndComp
 $Comp
-L +5V #PWR?
+L +5V #PWR032
 U 1 1 52FD5C6A
 P 8200 2100
-F 0 "#PWR?" H 8200 2190 20  0001 C CNN
+F 0 "#PWR032" H 8200 2190 20  0001 C CNN
 F 1 "+5V" H 8200 2190 30  0000 C CNN
 F 2 "" H 8200 2100 60  0000 C CNN
@@
 $EndComp
 $Comp
-L +12V #PWR?
+L +12V #PWR033
 U 1 1 52FD5C81
 P 2100 2950
-F 0 "#PWR?" H 2100 2900 20  0001 C CNN
+F 0 "#PWR033" H 2100 2900 20  0001 C CNN
 F 1 "+12V" H 2100 3050 30  0000 C CNN
 F 2 "" H 2100 2950 60  0000 C CNN
@@
 $EndComp
 $Comp
-L -12V #PWR?
+L -12V #PWR034
 U 1 1 52FD5C87
 P 2100 4450
-F 0 "#PWR?" H 2100 4580 20  0001 C CNN
+F 0 "#PWR034" H 2100 4580 20  0001 C CNN
 F 1 "-12V" H 2100 4550 30  0000 C CNN
 F 2 "" H 2100 4450 60  0000 C CNN
@@
 $EndComp
 $Comp
-L LM317 U?
+L LM317 U9
 U 1 1 52FD5C9C
 P 2950 6000
-F 0 "U?" H 2950 6300 60  0000 C CNN
+F 0 "U9" H 2950 6300 60  0000 C CNN
 F 1 "LM317" H 3000 5750 60  0000 L CNN
 F 2 "~" H 2950 6000 60  0000 C CNN
@@
 $EndComp
 $Comp
-L JUMPER JP?
+L JUMPER JP2
 U 1 1 52FD5CC4
 P 2950 2550
-F 0 "JP?" H 2950 2700 60  0000 C CNN
+F 0 "JP2" H 2950 2700 60  0000 C CNN
 F 1 "JUMPER" H 2950 2470 40  0000 C CNN
 F 2 "~" H 2950 2550 60  0000 C CNN
@@
 $EndComp
 $Comp
-L JUMPER JP?
+L JUMPER JP3
 U 1 1 52FD5CD1
 P 2950 4950
-F 0 "JP?" H 2950 5100 60  0000 C CNN
+F 0 "JP3" H 2950 5100 60  0000 C CNN
 F 1 "JUMPER" H 2950 4870 40  0000 C CNN
 F 2 "~" H 2950 4950 60  0000 C CNN
@@
 $EndComp
 $Comp
-L JUMPER JP?
+L JUMPER JP1
 U 1 1 52FD5CE8
 P 1050 3600
-F 0 "JP?" H 1050 3750 60  0000 C CNN
+F 0 "JP1" H 1050 3750 60  0000 C CNN
 F 1 "JUMPER" H 1050 3520 40  0000 C CNN
 F 2 "~" H 1050 3600 60  0000 C CNN
@@
 $EndComp
 $Comp
-L GND #PWR?
+L GND #PWR035
 U 1 1 52FD5CF0
 P 750 3850
-F 0 "#PWR?" H 750 3850 30  0001 C CNN
+F 0 "#PWR035" H 750 3850 30  0001 C CNN
 F 1 "GND" H 750 3780 30  0001 C CNN
 F 2 "" H 750 3850 60  0000 C CNN
@@
 $EndComp
 $Comp
-L AGND #PWR?
+L AGND #PWR036
 U 1 1 52FD5CFF
 P 1350 3850
-F 0 "#PWR?" H 1350 3850 40  0001 C CNN
+F 0 "#PWR036" H 1350 3850 40  0001 C CNN
 F 1 "AGND" H 1350 3780 50  0000 C CNN
 F 2 "" H 1350 3850 60  0000 C CNN
@@
 $EndComp
 $Comp
-L AGND #PWR?
+L AGND #PWR037
 U 1 1 52FD5D46
 P 1850 3900
-F 0 "#PWR?" H 1850 3900 40  0001 C CNN
+F 0 "#PWR037" H 1850 3900 40  0001 C CNN
 F 1 "AGND" H 1850 3830 50  0000 C CNN
 F 2 "" H 1850 3900 60  0000 C CNN
@@
 $EndComp
 $Comp
-L FE_V+ #PWR?
+L FE_V+ #PWR038
 U 1 1 52FD5DC4
 P 3550 2400
-F 0 "#PWR?" H 3550 2500 30  0001 C CNN
+F 0 "#PWR038" H 3550 2500 30  0001 C CNN
 F 1 "FE_V+" H 3550 2500 30  0000 C CNN
 F 2 "" H 3550 2400 60  0000 C CNN
@@
 $EndComp
 $Comp
-L FE_V- #PWR?
+L FE_V- #PWR39
 U 1 1 52FD5DD3
 P 3550 5100
-F 0 "#PWR?" H 3550 5300 40  0001 C CNN
+F 0 "#PWR39" H 3550 5300 40  0001 C CNN
 F 1 "FE_V-" H 3550 5250 40  0000 C CNN
 F 2 "" H 3550 5100 60  0000 C CNN
@@
 $EndComp
 $Comp
-L LM7812 U?
+L LM7812 U7
 U 1 1 52FD5E19
 P 2950 3250
-F 0 "U?" H 3100 3054 60  0000 C CNN
+F 0 "U7" H 3100 3054 60  0000 C CNN
 F 1 "LM7812" H 2950 3450 60  0000 C CNN
 F 2 "~" H 2950 3250 60  0000 C CNN
@@
 $EndComp
 $Comp
-L LM7812 U?
+L LM7812 U8
 U 1 1 52FD5E44
 P 2950 4250
-F 0 "U?" H 3100 4054 60  0000 C CNN
+F 0 "U8" H 3100 4054 60  0000 C CNN
 F 1 "LM7812" H 2950 4450 60  0000 C CNN
 F 2 "~" H 2950 4250 60  0000 C CNN
@@
 $EndComp
 $Comp
-L R R?
+L R R17
 U 1 1 52FD5E88
 P 3950 5150
-F 0 "R?" V 4030 5150 40  0000 C CNN
+F 0 "R17" V 4030 5150 40  0000 C CNN
 F 1 "R" V 3957 5151 40  0000 C CNN
 F 2 "~" V 3880 5150 30  0000 C CNN
@@
 $EndComp
 $Comp
-L AGND #PWR?
+L AGND #PWR039
 U 1 1 52FD5EA1
 P 4300 5000
-F 0 "#PWR?" H 4300 5000 40  0001 C CNN
+F 0 "#PWR039" H 4300 5000 40  0001 C CNN
 F 1 "AGND" H 4300 4930 50  0000 C CNN
 F 2 "" H 4300 5000 60  0000 C CNN
@@
 $EndComp
 $Comp
-L LM317 U?
+L LM317 U6
 U 1 1 52FD5F2E
 P 2950 1550
-F 0 "U?" H 2950 1850 60  0000 C CNN
+F 0 "U6" H 2950 1850 60  0000 C CNN
 F 1 "LM317" H 3000 1300 60  0000 L CNN
 F 2 "~" H 2950 1550 60  0000 C CNN
@@
 $EndComp
 $Comp
-L R R?
+L R R16
 U 1 1 52FD5F36
 P 3950 2400
-F 0 "R?" V 4030 2400 40  0000 C CNN
+F 0 "R16" V 4030 2400 40  0000 C CNN
 F 1 "R" V 3957 2401 40  0000 C CNN
 F 2 "~" V 3880 2400 30  0000 C CNN
@@
 $EndComp
 $Comp
-L AGND #PWR?
+L AGND #PWR040
 U 1 1 52FD5F42
 P 3950 2800
-F 0 "#PWR?" H 3950 2800 40  0001 C CNN
+F 0 "#PWR040" H 3950 2800 40  0001 C CNN
 F 1 "AGND" H 3950 2730 50  0000 C CNN
 F 2 "" H 3950 2800 60  0000 C CNN
@@
 V-_CURRENT_MON
 $Comp
-L R R?
+L R R21
 U 1 1 52FE6EC3
 P 5350 2350
-F 0 "R?" V 5430 2350 40  0000 C CNN
+F 0 "R21" V 5430 2350 40  0000 C CNN
 F 1 "R" V 5357 2351 40  0000 C CNN
 F 2 "~" V 5280 2350 30  0000 C CNN
@@
 $EndComp
 $Comp
-L R R?
+L R R22
 U 1 1 52FE6ED0
 P 5350 3050
-F 0 "R?" V 5430 3050 40  0000 C CNN
+F 0 "R22" V 5430 3050 40  0000 C CNN
 F 1 "R" V 5357 3051 40  0000 C CNN
 F 2 "~" V 5280 3050 30  0000 C CNN
@@
 Connection ~ 2950 3600
 $Comp
-L R R?
+L R R23
 U 1 1 52FE6F75
 P 5350 4250
-F 0 "R?" V 5430 4250 40  0000 C CNN
+F 0 "R23" V 5430 4250 40  0000 C CNN
 F 1 "R" V 5357 4251 40  0000 C CNN
 F 2 "~" V 5280 4250 30  0000 C CNN
@@
 	8200 2500 8850 2500
 $Comp
-L R R?
+L R R19
 U 1 1 52FE71B1
 P 4600 6150
-F 0 "R?" V 4680 6150 40  0000 C CNN
+F 0 "R19" V 4680 6150 40  0000 C CNN
 F 1 "R" V 4607 6151 40  0000 C CNN
 F 2 "~" V 4530 6150 30  0000 C CNN
@@
 V-_MON
 $Comp
-L R R?
+L R R20
 U 1 1 52FE73F0
 P 4650 1400
-F 0 "R?" V 4730 1400 40  0000 C CNN
+F 0 "R20" V 4730 1400 40  0000 C CNN
 F 1 "R" V 4657 1401 40  0000 C CNN
 F 2 "~" V 4580 1400 30  0000 C CNN
@@
 V+_MON
 $Comp
-L LM324 U?
-U 1 1 52FE778A
+L LM324 U10
+U 2 1 52FE778A
 P 8250 5950
-F 0 "U?" H 8300 6150 60  0000 C CNN
+F 0 "U10" H 8300 6150 60  0000 C CNN
 F 1 "LM324" H 8400 5750 50  0000 C CNN
 F 2 "" H 8250 5950 60  0000 C CNN
 F 3 "" H 8250 5950 60  0000 C CNN
-	1    8250 5950
-	1    0    0    -1
-$EndComp
-$Comp
-L +12V #PWR?
+	2    8250 5950
+	1    0    0    -1
+$EndComp
+$Comp
+L +12V #PWR041
 U 1 1 52FE7790
 P 8150 5350
-F 0 "#PWR?" H 8150 5300 20  0001 C CNN
+F 0 "#PWR041" H 8150 5300 20  0001 C CNN
 F 1 "+12V" H 8150 5450 30  0000 C CNN
 F 2 "" H 8150 5350 60  0000 C CNN
@@
 $EndComp
 $Comp
-L -12V #PWR?
+L -12V #PWR042
 U 1 1 52FE7796
 P 8150 6500
-F 0 "#PWR?" H 8150 6630 20  0001 C CNN
+F 0 "#PWR042" H 8150 6630 20  0001 C CNN
 F 1 "-12V" H 8150 6600 30  0000 C CNN
 F 2 "" H 8150 6500 60  0000 C CNN
@@
 	8150 5550 8150 5350
 $Comp
-L LM324 U?
+L LM324 U10
 U 1 1 52FE784E
 P 8250 4250
-F 0 "U?" H 8300 4450 60  0000 C CNN
+F 0 "U10" H 8300 4450 60  0000 C CNN
 F 1 "LM324" H 8400 4050 50  0000 C CNN
 F 2 "" H 8250 4250 60  0000 C CNN
@@
 $EndComp
 $Comp
-L +12V #PWR?
+L +12V #PWR043
 U 1 1 52FE7854
 P 8150 3650
-F 0 "#PWR?" H 8150 3600 20  0001 C CNN
+F 0 "#PWR043" H 8150 3600 20  0001 C CNN
 F 1 "+12V" H 8150 3750 30  0000 C CNN
 F 2 "" H 8150 3650 60  0000 C CNN
@@
 $EndComp
 $Comp
-L -12V #PWR?
+L -12V #PWR044
 U 1 1 52FE785A
 P 8150 4800
-F 0 "#PWR?" H 8150 4930 20  0001 C CNN
+F 0 "#PWR044" H 8150 4930 20  0001 C CNN
 F 1 "-12V" H 8150 4900 30  0000 C CNN
 F 2 "" H 8150 4800 60  0000 C CNN
@@
 V+_MON
 $Comp
-L R R?
+L R R24
 U 1 1 52FE6F7B
 P 5350 4950
-F 0 "R?" V 5430 4950 40  0000 C CNN
+F 0 "R24" V 5430 4950 40  0000 C CNN
 F 1 "R" V 5357 4951 40  0000 C CNN
 F 2 "~" V 5280 4950 30  0000 C CNN
@@
 $EndComp
 $Comp
-L RVAR R?
+L RVAR R15
 U 1 1 52FE7AD6
 P 3950 1700
-F 0 "R?" V 4030 1650 50  0000 C CNN
+F 0 "R15" V 4030 1650 50  0000 C CNN
 F 1 "RVAR" V 3870 1760 50  0000 C CNN
 F 2 "~" H 3950 1700 60  0000 C CNN
@@
 $EndComp
 $Comp
-L RVAR R?
+L RVAR R18
 U 1 1 52FE7AE3
 P 3950 5850
-F 0 "R?" V 4030 5800 50  0000 C CNN
+F 0 "R18" V 4030 5800 50  0000 C CNN
 F 1 "RVAR" V 3870 5910 50  0000 C CNN
 F 2 "~" H 3950 5850 60  0000 C CNN
