File: benchbudee/PowerMonitor.sch (KiCad schematic (older format))
At the start: 18 parts, among them U10 LM324, U6 LM317, U7 LM7812, U8 LM7812, U9 LM317

Commit message: New blinky 4 project, mods to blinky and benchbudee for new version
Parts:
- R16, R17, R19, R20, R21, R22, R23, R24: symbol R -> R-RESCUE-benchbudee
- U10: symbol LM324 -> LM324-RESCUE-benchbudee
Changed lines of the file:
@@
 EESchema Schematic File Version 2
+LIBS:benchbudee-rescue
 LIBS:power
 LIBS:device
@@
 LIBS:memory
 LIBS:xilinx
-LIBS:special
 LIBS:microcontrollers
 LIBS:dsp
@@
 $EndDescr
 $Comp
-L +3.3V #PWR53
+L +3.3V-RESCUE-benchbudee #PWR53
 U 1 1 52FD5C63
 P 8400 2100
@@
 $EndComp
 $Comp
-L GND #PWR39
+L GND-RESCUE-benchbudee #PWR39
 U 1 1 52FD5CF0
 P 750 3850
@@
 $EndComp
 $Comp
-L R R17
+L R-RESCUE-benchbudee R17
 U 1 1 52FD5E88
 P 3950 5150
@@
 $EndComp
 $Comp
-L R R16
+L R-RESCUE-benchbudee R16
 U 1 1 52FD5F36
 P 3950 2400
@@
 V-_CURRENT_MON
 $Comp
-L R R21
+L R-RESCUE-benchbudee R21
 U 1 1 52FE6EC3
 P 5350 2350
@@
 $EndComp
 $Comp
-L R R22
+L R-RESCUE-benchbudee R22
 U 1 1 52FE6ED0
 P 5350 3050
@@
 Connection ~ 2950 3600
 $Comp
-L R R23
+L R-RESCUE-benchbudee R23
 U 1 1 52FE6F75
 P 5350 4250
@@
 	8200 2500 8850 2500
 $Comp
-L R R19
+L R-RESCUE-benchbudee R19
 U 1 1 52FE71B1
 P 4600 6150
@@
 V-_MON
 $Comp
-L R R20
+L R-RESCUE-benchbudee R20
 U 1 1 52FE73F0
 P 4650 1400
@@
 V+_MON
 $Comp
-L LM324 U10
+L LM324-RESCUE-benchbudee U10
 U 2 1 52FE778A
 P 8250 5550
@@
 	8150 5150 8150 4950
 $Comp
-L LM324 U10
+L LM324-RESCUE-benchbudee U10
 U 1 1 52FE784E
 P 8250 3900
@@
 V+_MON
 $Comp
-L R R24
+L R-RESCUE-benchbudee R24
 U 1 1 52FE6F7B
 P 5350 4950
