File: benchbudee/Arduino.sch (KiCad schematic (older format))
At the start: 20 parts

Commit message: New blinky 4 project, mods to blinky and benchbudee for new version
Parts:
- R27, R28, R29, R30, R31, R32, R33, R34, R35, R36, R37, R38, R39, R40, R41, R42, R43, R46, R47: symbol R -> R-RESCUE-benchbudee
Changed lines of the file:
@@
 EESchema Schematic File Version 2
+LIBS:benchbudee-rescue
 LIBS:power
 LIBS:device
@@
 LIBS:memory
 LIBS:xilinx
-LIBS:special
 LIBS:microcontrollers
 LIBS:dsp
@@
 CURR_MEAS
 $Comp
-L R R38
+L R-RESCUE-benchbudee R38
 U 1 1 53206503
 P 7150 3200
@@
 	7400 3200 7600 3200
 $Comp
-L R R42
+L R-RESCUE-benchbudee R42
 U 1 1 53206A18
 P 7150 4550
@@
 	7400 4550 7600 4550
 $Comp
-L GND #PWR70
+L GND-RESCUE-benchbudee #PWR70
 U 1 1 53206A3A
 P 8650 4900
@@
 	8650 4550 8650 4900
 $Comp
-L R R34
+L R-RESCUE-benchbudee R34
 U 1 1 53206A58
 P 4300 3500
@@
 $EndComp
 $Comp
-L R R33
+L R-RESCUE-benchbudee R33
 U 1 1 53206A63
 P 4300 3350
@@
 V-_ADJ_MON
 $Comp
-L R R32
+L R-RESCUE-benchbudee R32
 U 1 1 53207FED
 P 4300 3200
@@
 $EndComp
 $Comp
-L R R31
+L R-RESCUE-benchbudee R31
 U 1 1 53207FF8
 P 4300 3050
@@
 	4700 3200 4550 3200
 $Comp
-L R R35
+L R-RESCUE-benchbudee R35
 U 1 1 5320805A
 P 7150 2750
@@
 $EndComp
 $Comp
-L R R36
+L R-RESCUE-benchbudee R36
 U 1 1 53208065
 P 7150 2900
@@
 $EndComp
 $Comp
-L R R37
+L R-RESCUE-benchbudee R37
 U 1 1 53208070
 P 7150 3050
@@
 $EndComp
 $Comp
-L R R41
+L R-RESCUE-benchbudee R41
 U 1 1 5320807B
 P 7150 3650
@@
 LED_EN_PWM
 $Comp
-L R R39
+L R-RESCUE-benchbudee R39
 U 1 1 53208124
 P 7150 3350
@@
 TC_CS_N
 $Comp
-L R R40
+L R-RESCUE-benchbudee R40
 U 1 1 532188BC
 P 7150 3500
@@
 FAN_MODE
 $Comp
-L R R43
+L R-RESCUE-benchbudee R43
 U 1 1 53262459
 P 7150 4700
@@
 	6900 4700 6700 4700
 $Comp
-L R R30
+L R-RESCUE-benchbudee R30
 U 1 1 532624A4
 P 4300 2900
@@
 	3150 2300 3150 2450
 $Comp
-L GND #PWR69
+L GND-RESCUE-benchbudee #PWR69
 U 1 1 5356A2E7
 P 3600 2750
@@
 $EndComp
 $Comp
-L R R28
+L R-RESCUE-benchbudee R28
 U 1 1 5356A2F9
 P 4300 2600
@@
 $EndComp
 $Comp
-L R R29
+L R-RESCUE-benchbudee R29
 U 1 1 5356A304
 P 4300 2750
@@
 $EndComp
 $Comp
-L R R27
+L R-RESCUE-benchbudee R27
 U 1 1 5356A30F
 P 4300 2450
@@
 ~RESET
 $Comp
-L R R46
+L R-RESCUE-benchbudee R46
 U 1 1 535F6093
 P 7150 3950
@@
 ~DR
 $Comp
-L R R47
+L R-RESCUE-benchbudee R47
 U 1 1 535F609C
 P 7150 4100
