File: benchbudee/Fan.sch (KiCad schematic (older format))
At the start: 18 parts, among them Q2 MOSFET_N, Q3 MOSFET_N, Q4 MOSFET_N, Q5 MOSFET_N, Q6 MOSFET_N, Q7 MOSFET_N, U11 MCP4922-E/P, U12 MCP4922-E/P, U13 OPA4170, U4 OPA4170

Commit message: New blinky 4 project, mods to blinky and benchbudee for new version
Parts:
- R25, R26, R48, R49: symbol R -> R-RESCUE-benchbudee
- U11, U12: symbol MCP4922-E/P -> MCP4922-E/P-RESCUE-benchbudee
- U13, U4: symbol LM324 -> LM324-RESCUE-benchbudee
Changed lines of the file:
@@
 EESchema Schematic File Version 2
+LIBS:benchbudee-rescue
 LIBS:power
 LIBS:device
@@
 LIBS:memory
 LIBS:xilinx
-LIBS:special
 LIBS:microcontrollers
 LIBS:dsp
@@
 FAN_PWM
 $Comp
-L LM324 U4
+L LM324-RESCUE-benchbudee U4
 U 2 1 52FBCCEC
 P 7300 2850
@@
 $EndComp
 $Comp
-L MCP4922-E/P U11
+L MCP4922-E/P-RESCUE-benchbudee U11
 U 1 1 52FBCE6B
 P 3850 2900
@@
 CURR_MEAS
 $Comp
-L R R25
+L R-RESCUE-benchbudee R25
 U 1 1 52FBCF5F
 P 4900 2750
@@
 $EndComp
 $Comp
-L R R26
+L R-RESCUE-benchbudee R26
 U 1 1 532608E6
 P 8750 4250
@@
 FAN_PWM
 $Comp
-L LM324 U13
+L LM324-RESCUE-benchbudee U13
 U 1 1 53626B76
 P -44900 -84300
@@
 $EndComp
 $Comp
-L MCP4922-E/P U12
+L MCP4922-E/P-RESCUE-benchbudee U12
 U 1 1 53626B8E
 P -48350 -84250
@@
 CURR_MEAS
 $Comp
-L R R48
+L R-RESCUE-benchbudee R48
 U 1 1 53626B95
 P -47300 -84400
@@
 $EndComp
 $Comp
-L R R49
+L R-RESCUE-benchbudee R49
 U 1 1 53626BC4
 P -43450 -82900
