File: benchbudee/LED_Driver.sch (KiCad schematic (older format))
At the start: 6 parts, among them U5 AP5726

Commit message: New blinky 4 project, mods to blinky and benchbudee for new version
Parts:
- C4, C5: symbol C -> C-RESCUE-benchbudee
- R14: symbol R -> R-RESCUE-benchbudee
Changed lines of the file:
@@
 EESchema Schematic File Version 2
+LIBS:benchbudee-rescue
 LIBS:power
 LIBS:device
@@
 LIBS:memory
 LIBS:xilinx
-LIBS:special
 LIBS:microcontrollers
 LIBS:dsp
@@
 $EndComp
 $Comp
-L GND #PWR36
+L GND-RESCUE-benchbudee #PWR36
 U 1 1 52FF5DCE
 P 3500 2850
@@
 $EndComp
 $Comp
-L C C4
+L C-RESCUE-benchbudee C4
 U 1 1 52FF5DF1
 P 3500 2500
@@
 	8700 2200 8700 2400
 $Comp
-L C C5
+L C-RESCUE-benchbudee C5
 U 1 1 52FF5E7B
 P 8700 2600
@@
 $EndComp
 $Comp
-L GND #PWR37
+L GND-RESCUE-benchbudee #PWR37
 U 1 1 52FF5E88
 P 4650 4100
@@
 $EndComp
 $Comp
-L GND #PWR38
+L GND-RESCUE-benchbudee #PWR38
 U 1 1 52FF5E8E
 P 8700 3050
@@
 Connection ~ 5750 2200
 $Comp
-L R R14
+L R-RESCUE-benchbudee R14
 U 1 1 52FF5EC9
 P 5750 3650
