File: benchbudee/Relay.sch (KiCad schematic (older format))
At the start: 11 parts, among them K1 1461069-5, Q1 2N3904, U1 LTV-816S

Commit message: New blinky 4 project, mods to blinky and benchbudee for new version
Parts:
- D1: symbol LED -> LED-RESCUE-benchbudee
- R1, R2, R3, R4, R5, R6: symbol R -> R-RESCUE-benchbudee
Changed lines of the file:
@@
 EESchema Schematic File Version 2
+LIBS:benchbudee-rescue
 LIBS:power
 LIBS:device
@@
 LIBS:memory
 LIBS:xilinx
-LIBS:special
 LIBS:microcontrollers
 LIBS:dsp
@@
 RELAY-
 $Comp
-L R R4
+L R-RESCUE-benchbudee R4
 U 1 1 52FBF34F
 P 6650 3900
@@
 $EndComp
 $Comp
-L LED D1
+L LED-RESCUE-benchbudee D1
 U 1 1 52FBF377
 P 6100 4200
@@
 	7450 3200 7450 3700
 $Comp
-L R R6
+L R-RESCUE-benchbudee R6
 U 1 1 52FBFB64
 P 7450 4450
@@
 	7450 4100 7450 4200
 $Comp
-L GND #PWR19
+L GND-RESCUE-benchbudee #PWR19
 U 1 1 52FBFB7C
 P 7450 5100
@@
 	7450 4700 7450 5100
 $Comp
-L R R2
+L R-RESCUE-benchbudee R2
 U 1 1 52FBFBA4
 P 6100 4750
@@
 	6100 4500 6100 4400
 $Comp
-L GND #PWR17
+L GND-RESCUE-benchbudee #PWR17
 U 1 1 52FBFBD1
 P 6100 5100
@@
 	6100 5000 6100 5100
 $Comp
-L R R3
+L R-RESCUE-benchbudee R3
 U 1 1 52FBFC4A
 P 6600 2650
@@
 	6600 3100 4850 3100
 $Comp
-L R R1
+L R-RESCUE-benchbudee R1
 U 1 1 52FBFCE0
 P 3200 3400
@@
 	7050 3550 7050 3600
 $Comp
-L R R5
+L R-RESCUE-benchbudee R5
 U 1 1 535DB520
 P 7050 2650
