File: benchbudee/Thermocouple.sch (KiCad schematic (older format))
At the start: 21 parts, among them P2 CONN_2, P3 CONN_3X2, U2 MCP3901, U3 LMT84, U4 OPA4170

Commit message: New blinky 4 project, mods to blinky and benchbudee for new version
Parts:
- C10, C6, C7, C8, C9: symbol C -> C-RESCUE-benchbudee
- R10, R11, R12, R13, R44, R45, R50, R51, R7, R8, R9: symbol R -> R-RESCUE-benchbudee
- U4: symbol LM324 -> LM324-RESCUE-benchbudee
Changed lines of the file:
@@
 EESchema Schematic File Version 2
+LIBS:benchbudee-rescue
 LIBS:power
 LIBS:device
@@
 LIBS:memory
 LIBS:xilinx
-LIBS:special
 LIBS:microcontrollers
 LIBS:dsp
@@
 ~CS
 $Comp
-L LM324 U4
+L LM324-RESCUE-benchbudee U4
 U 3 1 52FAF263
 P 7650 2200
@@
 $EndComp
 $Comp
-L LM324 U4
+L LM324-RESCUE-benchbudee U4
 U 4 1 52FAF27A
 P 7650 4300
@@
 $EndComp
 $Comp
-L LM324 U4
+L LM324-RESCUE-benchbudee U4
 U 1 1 52FAF280
 P 5500 3250
@@
 $EndComp
 $Comp
-L R R12
+L R-RESCUE-benchbudee R12
 U 1 1 52FAF2B2
 P 9350 3750
@@
 $EndComp
 $Comp
-L R R11
+L R-RESCUE-benchbudee R11
 U 1 1 52FAF2BF
 P 7000 2600
@@
 $EndComp
 $Comp
-L R R13
+L R-RESCUE-benchbudee R13
 U 1 1 52FAF2CF
 P 7000 3900
@@
 $EndComp
 $Comp
-L R R9
+L R-RESCUE-benchbudee R9
 U 1 1 52FAF2EA
 P 6450 2200
@@
 $EndComp
 $Comp
-L R R7
+L R-RESCUE-benchbudee R7
 U 1 1 52FAF2F0
 P 5350 2200
@@
 $EndComp
 $Comp
-L R R8
+L R-RESCUE-benchbudee R8
 U 1 1 52FAF2F6
 P 5400 4300
@@
 $EndComp
 $Comp
-L R R10
+L R-RESCUE-benchbudee R10
 U 1 1 52FAF2FC
 P 6450 4300
@@
 $EndComp
 $Comp
-L R R44
+L R-RESCUE-benchbudee R44
 U 1 1 535EDF39
 P 9600 3750
@@
 $EndComp
 $Comp
-L R R45
+L R-RESCUE-benchbudee R45
 U 1 1 535EDF44
 P 9850 3750
@@
 	5700 4800 5700 4950
 $Comp
-L C C10
+L C-RESCUE-benchbudee C10
 U 1 1 535EFF7B
 P 6250 5550
@@
 Connection ~ 5700 6350
 $Comp
-L C C9
+L C-RESCUE-benchbudee C9
 U 1 1 535F003F
 P 5300 3800
@@
 $EndComp
 $Comp
-L C C8
+L C-RESCUE-benchbudee C8
 U 1 1 535F004A
 P 5300 2700
@@
 	3200 1450 3200 1800
 $Comp
-L C C7
+L C-RESCUE-benchbudee C7
 U 1 1 535F0A37
 P 3550 1550
@@
 	3200 1550 3350 1550
 $Comp
-L C C6
+L C-RESCUE-benchbudee C6
 U 1 1 535F0E29
 P 2450 1550
@@
 	4850 3800 4850 3400
 $Comp
-L R R51
+L R-RESCUE-benchbudee R51
 U 1 1 5362AFBB
 P 4850 4050
@@
 	4850 4300 4850 4500
 $Comp
-L R R50
+L R-RESCUE-benchbudee R50
 U 1 1 5362B033
 P 4400 5750
