File: blinky4/blinky4.kicad_pcb (KiCad board)
At the start: 2 copper layers, 38.1 x 35.6 mm, 7 parts, among them U1 7555

Commit message: Finished version of Getting to Blinky v4
Parts:
- moved R3 1.27 mm to (149.9, 106.7), turned to 270 degrees
- turned C1 to 270 degrees
Connections:
- U1 pad 5: GND -> Net-(U1-Pad5)
Routing:
- net /VDD: track 0.00 -> 17.0 mm, vias 0 -> 2
- net Net-(C1-Pad1): track 0.00 -> 15.3 mm
- net Net-(R1-Pad2): track 0.00 -> 10.7 mm
- net Net-(R3-Pad1): track 0.00 -> 6.49 mm
- net Net-(D1-Pad2): track 0.00 -> 3.95 mm
- net GND: track 0.00 -> 3.81 mm, vias 0 -> 1
- added copper zone on B.Cu, net /VDD
- added copper zone on F.Cu, net GND
Other:
- net class Default: clearance 0.2 -> 0.254; trace_width 0.25 -> 0.254; via_dia 0.6 -> 0.6858; via_drill 0.4 -> 0.3302
- rule trace_clearance: 0.2 -> 0.254
- rule trace_min: 0.2 -> 0.1524
- rule via_min_drill: 0.3 -> 0.3302
- rule via_min_size: 0.4 -> 0.6858
- board text added: "Getting to Blinky v4"
Changed lines of the file:
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@@
 (kicad_pcb (version 4) (host pcbnew 4.0.3-stable)
   (general
-    (links 15)
-    (no_connects 15)
-    (area 0 0 0 0)
+    (links 14)
+    (no_connects 0)
+    (area 139.624999 88.824999 177.875001 124.535001)
     (thickness 1.6)
-    (drawings 4)
-    (tracks 0)
+    (drawings 5)
+    (tracks 26)
     (zones 0)
     (modules 7)
-    (nets 7)
+    (nets 8)
   )
   (page A4)
   (layers
     (0 F.Cu signal)
-    (31 B.Cu signal)
+    (31 B.Cu signal hide)
     (32 B.Adhes user)
     (33 F.Adhes user)
@@
   )
   (setup
-    (last_trace_width 0.25)
-    (trace_clearance 0.2)
+    (last_trace_width 0.254)
+    (trace_clearance 0.254)
     (zone_clearance 0.508)
     (zone_45_only no)
-    (trace_min 0.2)
+    (trace_min 0.1524)
     (segment_width 0.2)
     (edge_width 0.15)
-    (via_size 0.6)
-    (via_drill 0.4)
-    (via_min_size 0.4)
-    (via_min_drill 0.3)
+    (via_size 0.6858)
+    (via_drill 0.3302)
+    (via_min_size 0.6858)
+    (via_min_drill 0.3302)
     (uvia_size 0.3)
     (uvia_drill 0.1)
@@
     (visible_elements FFFFFF7F)
     (pcbplotparams
-      (layerselection 0x00030_80000001)
-      (usegerberextensions false)
+      (layerselection 0x010f0_80000001)
+      (usegerberextensions true)
       (excludeedgelayer true)
       (linewidth 0.100000)
@@
       (psa4output false)
       (plotreference true)
-      (plotvalue true)
+      (plotvalue false)
       (plotinvisibletext false)
       (padsonsilk false)
-      (subtractmaskfromsilk false)
+      (subtractmaskfromsilk true)
       (outputformat 1)
       (mirror false)
-      (drillshape 1)
+      (drillshape 0)
       (scaleselection 1)
-      (outputdirectory ""))
+      (outputdirectory gerbers/))
   )
   (net 0 "")
@@
   (net 5 "Net-(R1-Pad2)")
   (net 6 "Net-(R3-Pad1)")
+  (net 7 "Net-(U1-Pad5)")
   (net_class Default "This is the default net class."
-    (clearance 0.2)
-    (trace_width 0.25)
-    (via_dia 0.6)
-    (via_drill 0.4)
+    (clearance 0.254)
+    (trace_width 0.254)
+    (via_dia 0.6858)
+    (via_drill 0.3302)
     (uvia_dia 0.3)
     (uvia_drill 0.1)
@@
     (add_net "Net-(R1-Pad2)")
     (add_net "Net-(R3-Pad1)")
+    (add_net "Net-(U1-Pad5)")
   )
   (module Capacitors_SMD:C_1206_HandSoldering (layer F.Cu)
-    (at 166.37 111.76 90)
+    (at 166.37 111.76 270)
     (descr "Capacitor SMD 1206, hand soldering")
     (tags "capacitor 1206")
     (attr smd)
-    (fp_text reference C1 (at 0 -2.3 90) (layer F.SilkS)
-      (effects (font (size 1 1) (thickness 0.15)))
-    )
-    (fp_text value 1u (at 0 2.3 90) (layer F.Fab)
+    (fp_text reference C1 (at 2.54 -2.54 360) (layer F.SilkS)
+      (effects (font (size 1 1) (thickness 0.15)))
+    )
+    (fp_text value 1u (at 0 2.3 270) (layer F.Fab)
       (effects (font (size 1 1) (thickness 0.15)))
     )
@@
     (fp_line (start 1 -1.025) (end -1 -1.025) (layer F.SilkS) (width 0.15))
     (fp_line (start -1 1.025) (end 1 1.025) (layer F.SilkS) (width 0.15))
-    (pad 1 smd rect (at -2 0 90) (size 2 1.6) (layers F.Cu F.Paste F.Mask)
+    (pad 1 smd rect (at -2 0 270) (size 2 1.6) (layers F.Cu F.Paste F.Mask)
       (net 1 "Net-(C1-Pad1)"))
-    (pad 2 smd rect (at 2 0 90) (size 2 1.6) (layers F.Cu F.Paste F.Mask)
+    (pad 2 smd rect (at 2 0 270) (size 2 1.6) (layers F.Cu F.Paste F.Mask)
       (net 2 GND))
     (model Capacitors_SMD.3dshapes/C_1206_HandSoldering.wrl
@@
     (tags "LED 0805 SMD")
     (attr smd)
-    (fp_text reference D1 (at 0 -1.75 90) (layer F.SilkS)
+    (fp_text reference D1 (at 1.27 2.54 180) (layer F.SilkS)
       (effects (font (size 1 1) (thickness 0.15)))
     )
@@
     (tags "resistor 0805")
     (attr smd)
-    (fp_text reference R1 (at 0 -2.1 270) (layer F.SilkS)
+    (fp_text reference R1 (at -2.54 -2.54 360) (layer F.SilkS)
       (effects (font (size 1 1) (thickness 0.15)))
     )
@@
     (tags "resistor 0805")
     (attr smd)
-    (fp_text reference R2 (at 0 -2.1 270) (layer F.SilkS)
+    (fp_text reference R2 (at -2.54 -2.54 360) (layer F.SilkS)
       (effects (font (size 1 1) (thickness 0.15)))
     )
@@
   )
   (module Resistors_SMD:R_0805_HandSoldering (layer F.Cu)
-    (at 149.86 105.41 90)
+    (at 149.86 106.68 270)
     (descr "Resistor SMD 0805, hand soldering")
     (tags "resistor 0805")
     (attr smd)
-    (fp_text reference R3 (at 0 -2.1 90) (layer F.SilkS)
-      (effects (font (size 1 1) (thickness 0.15)))
-    )
-    (fp_text value 1K (at 0 2.1 90) (layer F.Fab)
+    (fp_text reference R3 (at -2.54 -2.54 360) (layer F.SilkS)
+      (effects (font (size 1 1) (thickness 0.15)))
+    )
+    (fp_text value 1K (at 0 2.1 270) (layer F.Fab)
       (effects (font (size 1 1) (thickness 0.15)))
     )
@@
     (fp_line (start 0.6 0.875) (end -0.6 0.875) (layer F.SilkS) (width 0.15))
     (fp_line (start -0.6 -0.875) (end 0.6 -0.875) (layer F.SilkS) (width 0.15))
-    (pad 1 smd rect (at -1.35 0 90) (size 1.5 1.3) (layers F.Cu F.Paste F.Mask)
+    (pad 1 smd rect (at -1.35 0 270) (size 1.5 1.3) (layers F.Cu F.Paste F.Mask)
       (net 6 "Net-(R3-Pad1)"))
-    (pad 2 smd rect (at 1.35 0 90) (size 1.5 1.3) (layers F.Cu F.Paste F.Mask)
+    (pad 2 smd rect (at 1.35 0 270) (size 1.5 1.3) (layers F.Cu F.Paste F.Mask)
       (net 3 "Net-(D1-Pad2)"))
     (model Resistors_SMD.3dshapes/R_0805_HandSoldering.wrl
@@
       (net 4 /VDD))
     (pad 5 smd rect (at 2.7 1.905) (size 1.55 0.6) (layers F.Cu F.Paste F.Mask)
-      (net 2 GND))
+      (net 7 "Net-(U1-Pad5)"))
     (pad 6 smd rect (at 2.7 0.635) (size 1.55 0.6) (layers F.Cu F.Paste F.Mask)
       (net 1 "Net-(C1-Pad1)"))
@@
       (net 4 /VDD))
   )
+  (gr_text "Getting to Blinky v4" (at 152.4 91.44) (layer F.SilkS)
+    (effects (font (size 1.5 1.5) (thickness 0.3)))
+  )
   (gr_line (start 139.7 88.9) (end 177.8 88.9) (angle 90) (layer Edge.Cuts) (width 0.15))
   (gr_line (start 177.8 124.46) (end 139.7 124.46) (angle 90) (layer Edge.Cuts) (width 0.15))
   (gr_line (start 177.8 88.9) (end 177.8 124.46) (angle 90) (layer Edge.Cuts) (width 0.15))
   (gr_line (start 139.7 124.46) (end 139.7 88.9) (angle 90) (layer Edge.Cuts) (width 0.15))
+  (segment (start 159.385 106.045) (end 161.45 106.045) (width 0.254) (layer F.Cu) (net 1))
+  (segment (start 158.115 104.775) (end 159.385 106.045) (width 0.254) (layer F.Cu) (net 1))
+  (segment (start 156.05 104.775) (end 158.115 104.775) (width 0.254) (layer F.Cu) (net 1))
+  (segment (start 161.45 106.045) (end 164.465 106.045) (width 0.254) (layer F.Cu) (net 1))
+  (segment (start 165.02 105.49) (end 166.37 105.49) (width 0.254) (layer F.Cu) (net 1))
+  (segment (start 164.465 106.045) (end 165.02 105.49) (width 0.254) (layer F.Cu) (net 1))
+  (segment (start 166.37 105.49) (end 166.37 109.76) (width 0.254) (layer F.Cu) (net 1))
+  (segment (start 158.75 106.68) (end 158.75 110.49) (width 0.254) (layer B.Cu) (net 2))
+  (via (at 158.75 110.49) (size 0.6858) (drill 0.3302) (layers F.Cu B.Cu) (net 2))
+  (segment (start 149.86 108.03) (end 149.86 111.98098) (width 0.254) (layer F.Cu) (net 3))
+  (segment (start 156.05 107.315) (end 155.575 107.315) (width 0.254) (layer F.Cu) (net 4))
+  (segment (start 155.575 107.315) (end 153.67 109.22) (width 0.254) (layer F.Cu) (net 4))
+  (via (at 153.67 109.22) (size 0.6858) (drill 0.3302) (layers F.Cu B.Cu) (net 4))
+  (segment (start 161.45 103.505) (end 161.45 101.76) (width 0.254) (layer F.Cu) (net 4))
+  (via (at 161.29 101.6) (size 0.6858) (drill 0.3302) (layers F.Cu B.Cu) (net 4))
+  (segment (start 161.45 101.76) (end 161.29 101.6) (width 0.254) (layer F.Cu) (net 4))
+  (segment (start 161.45 103.505) (end 161.45 97.63) (width 0.254) (layer F.Cu) (net 4))
+  (segment (start 163.91 95.17) (end 166.37 95.17) (width 0.254) (layer F.Cu) (net 4))
+  (segment (start 161.45 97.63) (end 163.91 95.17) (width 0.254) (layer F.Cu) (net 4))
+  (segment (start 161.45 104.775) (end 163.195 104.775) (width 0.254) (layer F.Cu) (net 5))
+  (segment (start 165.18 102.79) (end 166.37 102.79) (width 0.254) (layer F.Cu) (net 5))
+  (segment (start 163.195 104.775) (end 165.18 102.79) (width 0.254) (layer F.Cu) (net 5))
+  (segment (start 166.37 97.87) (end 166.37 102.79) (width 0.254) (layer F.Cu) (net 5))
+  (segment (start 156.05 106.045) (end 153.035 106.045) (width 0.254) (layer F.Cu) (net 6))
+  (segment (start 152.32 105.33) (end 149.86 105.33) (width 0.254) (layer F.Cu) (net 6))
+  (segment (start 153.035 106.045) (end 152.32 105.33) (width 0.254) (layer F.Cu) (net 6))
+  (zone (net 2) (net_name GND) (layer F.Cu) (hatch edge 0.508)
+    (connect_pads (clearance 0.508))
+    (min_thickness 0.254)
+    (fill yes (arc_segments 16) (thermal_gap 0.508) (thermal_bridge_width 0.508))
+    (polygon
+      (pts
+        (xy 177.8 124.46) (xy 139.7 124.46) (xy 139.7 88.9) (xy 177.8 88.9)
+      )
+    )
+  )
+  (zone (net 4) (net_name /VDD) (layer B.Cu) (hatch edge 0.508)
+    (connect_pads (clearance 0.508))
+    (min_thickness 0.254)
+    (fill yes (arc_segments 16) (thermal_gap 0.508) (thermal_bridge_width 0.508))
+    (polygon
+      (pts
+        (xy 177.8 124.46) (xy 139.7 124.46) (xy 139.7 88.9) (xy 177.8 88.9)
+      )
+    )
+  )
 )
