File: blinky4/blinky4.sch (KiCad schematic (older format))
At the start: 7 parts, among them U1 7555

Commit message: Finished version of Getting to Blinky v4
Connections:
- wire segments 22 -> 21
Changed lines of the file:
@@
 Text Label 2850 3100 0    60   ~ 0
 VDD
-Wire Wire Line
-	5650 4700 5650 5300
-Connection ~ 5650 5300
 $EndSCHEMATC
